Commit message: Funcionando solo falange

File: scara/urdf/urdf.xacro (robot description, xacro)
@@ -55,5 +55,5 @@
     </link>
     <joint name="hombro" type="revolute">
-        <limit lower="-${pi/2}" upper="${pi/2}" effort="0.0" velocity="0.0"/>
+        <limit lower="-${pi}" upper="${pi}" effort="0.0" velocity="0.0"/>
         <origin xyz="0 0 0.5925" rpy="0 0 0" />
         <parent link="base_link" />
@@ -84,5 +84,5 @@
     </link>
     <joint name="codo" type="revolute">
-        <limit lower="-${pi/2}" upper="${pi/2}" effort="0.0" velocity="0.0"/>
+        <limit lower="-${pi}" upper="${pi}" effort="0.0" velocity="0.0"/>
         <origin xyz="0.4025 0 0" rpy="0 0 0" />
         <parent link="antebrazo" />
@@ -113,8 +113,8 @@
     </link>
     <joint name="falange" type="prismatic">
-        <origin xyz="0.37763 0 0.020231" rpy="0 0 0" />
+        <origin xyz="0.37763 0 0.170231" rpy="0 0 0" />
         <parent link="brazo" />
         <child link="mano" />
-        <axis xyz="0 0 1" />
+        <axis xyz="0 0 -1" />
         <limit lower="0" upper="0.15" effort="80" velocity="1" />
     </joint>

File: scara_hardware/config/ros2_control.xacro (robot description, xacro)
@@ -7,30 +7,30 @@
         <!-- Joint1 -->
         <param name="joint1_name">hombro</param>
-        <param name="joint1_controller_gain">1.0</param>
-        <param name="joint1_counts_per_unit">1000</param>
+        <param name="joint1_controller_gain">50.0</param>
+        <param name="joint1_counts_per_unit">186740.0</param>
         <param name="joint1_minimum_time_period">1</param>
-        <param name="joint1_maximum_time_period">10</param>
-        <param name="joint1_offset">10</param>
+        <param name="joint1_maximum_time_period">1000000</param>
+        <param name="joint1_offset">220000</param>
         <!-- Joint2 -->
         <param name="joint2_name">codo</param>
-        <param name="joint2_controller_gain">1.0</param>
-        <param name="joint2_counts_per_unit">1000</param>
-        <param name="joint2_minimum_time_period">1</param>
-        <param name="joint2_maximum_time_period">10</param>
-        <param name="joint2_offset">10</param>
+        <param name="joint2_controller_gain">50.0</param>
+        <param name="joint2_counts_per_unit">12308.0</param>
+        <param name="joint2_minimum_time_period">3</param>
+        <param name="joint2_maximum_time_period">1000000</param>
+        <param name="joint2_offset">-29000</param>
         <!-- Joint3 -->
         <param name="joint3_name">muneca</param>
-        <param name="joint3_controller_gain">1.0</param>
-        <param name="joint3_counts_per_unit">1000</param>
+        <param name="joint3_controller_gain">50.0</param>
+        <param name="joint3_counts_per_unit">1000.0</param>
         <param name="joint3_minimum_time_period">1</param>
-        <param name="joint3_maximum_time_period">10</param>
-        <param name="joint3_offset">10</param>
+        <param name="joint3_maximum_time_period">1000000</param>
+        <param name="joint3_offset">0</param>
         <!-- Joint4 -->
         <param name="joint4_name">falange</param>
-        <param name="joint4_controller_gain">1.0</param>
-        <param name="joint4_counts_per_unit">1000</param>
+        <param name="joint4_controller_gain">50.0</param>
+        <param name="joint4_counts_per_unit">1065200.0</param> <!-- 2 * 79890 / 0.15m -->
         <param name="joint4_minimum_time_period">1</param>
-        <param name="joint4_maximum_time_period">10</param>
-        <param name="joint4_offset">10</param>
+        <param name="joint4_maximum_time_period">1000000</param>
+        <param name="joint4_offset">0</param>
         <!-- Serial Communication -->
         <param name="loop_rate">30</param>
@@ -61,5 +61,5 @@
         <command_interface name="position"/>
         <state_interface name="position">
-          <param name="initial_value">0.0</param>
+          <param name="initial_value">0.1</param>
         </state_interface>
         <state_interface name="velocity">

Commit message: ¡¡¡¡¡Funciono!!!!!

File: scara/urdf/urdf.xacro (robot description, xacro)
@@ -55,5 +55,5 @@
     </link>
     <joint name="hombro" type="revolute">
-        <limit lower="-${pi}" upper="${pi}" effort="0.0" velocity="0.0"/>
+        <limit lower="-1.845" upper="1.845" effort="0.0" velocity="0.0"/>
         <origin xyz="0 0 0.5925" rpy="0 0 0" />
         <parent link="base_link" />
@@ -84,5 +84,5 @@
     </link>
     <joint name="codo" type="revolute">
-        <limit lower="-${pi}" upper="${pi}" effort="0.0" velocity="0.0"/>
+        <limit lower="-2.574" upper="2.574" effort="0.0" velocity="0.0"/>
         <origin xyz="0.4025 0 0" rpy="0 0 0" />
         <parent link="antebrazo" />

File: scara_hardware/config/ros2_control.xacro (robot description, xacro)
@@ -8,15 +8,15 @@
         <param name="joint1_name">hombro</param>
         <param name="joint1_controller_gain">50.0</param>
-        <param name="joint1_counts_per_unit">186740.0</param>
+        <param name="joint1_counts_per_unit">133005.464</param>
         <param name="joint1_minimum_time_period">1</param>
         <param name="joint1_maximum_time_period">1000000</param>
-        <param name="joint1_offset">220000</param>
+        <param name="joint1_offset">243400</param>
         <!-- Joint2 -->
         <param name="joint2_name">codo</param>
         <param name="joint2_controller_gain">50.0</param>
-        <param name="joint2_counts_per_unit">12308.0</param>
+        <param name="joint2_counts_per_unit">15481.74</param>
         <param name="joint2_minimum_time_period">3</param>
         <param name="joint2_maximum_time_period">1000000</param>
-        <param name="joint2_offset">-29000</param>
+        <param name="joint2_offset">-39850</param>
         <!-- Joint3 -->
         <param name="joint3_name">muneca</param>
@@ -43,5 +43,5 @@
         <command_interface name="position"/>
         <state_interface name="position">
-          <param name="initial_value">0.0</param>
+          <param name="initial_value">-1.84</param>
         </state_interface>
         <state_interface name="velocity">
@@ -52,5 +52,5 @@
         <command_interface name="position"/>
         <state_interface name="position">
-          <param name="initial_value">0.0</param>
+          <param name="initial_value">2.57</param>
         </state_interface>
         <state_interface name="velocity">
@@ -61,5 +61,5 @@
         <command_interface name="position"/>
         <state_interface name="position">
-          <param name="initial_value">0.1</param>
+          <param name="initial_value">0.0</param>
         </state_interface>
         <state_interface name="velocity">
